Commit message: Add visual frontier goal selection

File: src/active_3d_description/urdf/turtlebot3_burger.urdf (robot description, URDF)
Before this commit: robot turtlebot3_burger, 7 links, 6 joints
Links:
- added link ${namespace}explore_camera_link, mass 0.03; collision box size=0.035 0.055 0.030; visual box size=0.035 0.055 0.030
- added link ${namespace}explore_camera_optical_frame
Joints:
- added joint ${namespace}explore_camera_joint: type fixed, parent ${namespace}base_link, child ${namespace}explore_camera_link, origin xyz=0.055 0 0.190 rpy=0 0 0
- added joint ${namespace}explore_camera_optical_joint: type fixed, parent ${namespace}explore_camera_link, child ${namespace}explore_camera_optical_frame, origin xyz=0 0 0 rpy=-1.57079632679 0 -1.57079632679

Commit message: add isaac files

File: src/active_3d_description/urdf/turtlebot3_burger.urdf (robot description, URDF)
Before this commit: robot turtlebot3_burger, 9 links, 8 joints
Links:
- link ${namespace}base_link: geometry collision box size=0.140 0.140 0.143; visual mesh filename=/home/wanjunkim/ros2_project/3D-SLAM-with-Tilted-TurtleBot/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 scale=0.001 0.001 0.001
- link ${namespace}base_scan: geometry collision cylinder length=0.0315 radius=0.055; visual mesh filename=/home/wanjunkim/ros2_project/3D-SLAM-with-Tilted-TurtleBot/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 scale=0.001 0.001 0.001
- link ${namespace}wheel_left_link: geometry collision cylinder length=0.018 radius=0.033; visual mesh filename=/home/wanjunkim/ros2_project/3D-SLAM-with-Tilted-TurtleBot/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 scale=0.001 0.001 0.001
- link ${namespace}wheel_right_link: geometry collision cylinder length=0.018 radius=0.033; visual mesh filename=/home/wanjunkim/ros2_project/3D-SLAM-with-Tilted-TurtleBot/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 scale=0.001 0.001 0.001

File: src/active_3d_description/urdf/turtlebot3_waffle.urdf (robot description, URDF)
Before this commit: robot turtlebot3_waffle, 13 links, 12 joints
Links:
- link ${namespace}base_link: geometry collision box size=0.266 0.266 0.094; visual mesh filename=/home/wanjunkim/ros2_project/3D-SLAM-with-Tilted-TurtleBot/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 scale=0.001 0.001 0.001
- link ${namespace}base_scan: geometry collision cylinder length=0.0315 radius=0.055; visual mesh filename=/home/wanjunkim/ros2_project/3D-SLAM-with-Tilted-TurtleBot/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 scale=0.001 0.001 0.001
- link ${namespace}camera_link: geometry collision box size=0.012 0.132 0.020; visual mesh filename=/home/wanjunkim/ros2_project/3D-SLAM-with-Tilted-TurtleBot/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
- link ${namespace}wheel_left_link: geometry collision cylinder length=0.018 radius=0.033; visual mesh filename=/home/wanjunkim/ros2_project/3D-SLAM-with-Tilted-TurtleBot/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 scale=0.001 0.001 0.001
- link ${namespace}wheel_right_link: geometry collision cylinder length=0.018 radius=0.033; visual mesh filename=/home/wanjunkim/ros2_project/3D-SLAM-with-Tilted-TurtleBot/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 scale=0.001 0.001 0.001

File: src/active_3d_description/urdf/turtlebot3_waffle_pi.urdf (robot description, URDF)
Before this commit: robot turtlebot3_waffle_pi, 11 links, 10 joints
Links:
- link ${namespace}base_link: geometry collision box size=0.266 0.266 0.094; visual mesh filename=/home/wanjunkim/ros2_project/3D-SLAM-with-Tilted-TurtleBot/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 scale=0.001 0.001 0.001
- link ${namespace}base_scan: geometry collision cylinder length=0.0315 radius=0.055; visual mesh filename=/home/wanjunkim/ros2_project/3D-SLAM-with-Tilted-TurtleBot/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 scale=0.001 0.001 0.001
- link ${namespace}wheel_left_link: geometry collision cylinder length=0.018 radius=0.033; visual mesh filename=/home/wanjunkim/ros2_project/3D-SLAM-with-Tilted-TurtleBot/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 scale=0.001 0.001 0.001
- link ${namespace}wheel_right_link: geometry collision cylinder length=0.018 radius=0.033; visual mesh filename=/home/wanjunkim/ros2_project/3D-SLAM-with-Tilted-TurtleBot/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 scale=0.001 0.001 0.001

Commit message: final ver

File: src/active_3d_description/urdf/turtlebot3_burger.urdf (robot description, URDF)
Before this commit: robot turtlebot3_burger, 9 links, 8 joints
Links:
- link ${namespace}base_link: geometry collision box size=0.140 0.140 0.143; visual mesh filename=package://turtlebot3_description/meshes/bases/burger_base.s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 scale=0.001 0.001 0.001
- link ${namespace}base_scan: geometry collision cylinder length=0.0315 radius=0.055; visual mesh filename=package://turtlebot3_description/meshes/sensors/lds.stl scale=0.001 0.001 0.001
- link ${namespace}wheel_left_link: geometry collision cylinder length=0.018 radius=0.033; visual mesh filename=package://turtlebot3_description/meshes/wheels/left_tire.stl scale=0.001 0.001 0.001
- link ${namespace}wheel_right_link: geometry collision cylinder length=0.018 radius=0.033; visual mesh filename=package://turtlebot3_description/meshes/wheels/right_tire.s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 scale=0.001 0.001 0.001
